File: hardware/PRS.kicad_pcb (KiCad board)
At the start: 2 copper layers, 4 parts, among them K1 T9AS1D12-5, K2 T9AS1D12-5, K3 T9AS1D12-5, K4 T9AS1D12-5

Commit message: Commit
Parts:
- added D1: MMBD7000HC, Package_TO_SOT_SMD:SOT-23_Handsoldering, F.Cu at (98.8, 77.5)
- added D2: MMBD7000HC, Package_TO_SOT_SMD:SOT-23_Handsoldering, F.Cu at (132.1, 78.7)
- added D3: MMBD7000HC, Package_TO_SOT_SMD:SOT-23_Handsoldering, F.Cu at (162.6, 76.2)
- added D4: MMBD7000HC, Package_TO_SOT_SMD:SOT-23_Handsoldering, F.Cu at (199.4, 80.0)
- added D5: D_Zener, Diode_SMD:D_SMA_Handsoldering, F.Cu at (102.9, 111.8)
- added Q1: PMV37ENEA, Package_TO_SOT_SMD:SOT-23_Handsoldering, F.Cu at (108.0, 78.7)
- added Q2: PMV37ENEA, Package_TO_SOT_SMD:SOT-23_Handsoldering, F.Cu at (131.0, 88.0)
- added Q3: PMV37ENEA, Package_TO_SOT_SMD:SOT-23_Handsoldering, F.Cu at (163.8, 85.1)
- added Q4: PMV37ENEA, Package_TO_SOT_SMD:SOT-23_Handsoldering, F.Cu at (190.5, 77.5)
- added R1: 100k, Resistor_SMD:R_0603_1608Metric_Pad0.98x0.95mm_HandSolder, F.Cu at (99.1, 85.1)
- added R2: 100k, Resistor_SMD:R_0603_1608Metric_Pad0.98x0.95mm_HandSolder, F.Cu at (122.8, 85.1)
- added R3: 100k, Resistor_SMD:R_0603_1608Metric_Pad0.98x0.95mm_HandSolder, F.Cu at (167.3, 91.4)
- added R4: 100k, Resistor_SMD:R_0603_1608Metric_Pad0.98x0.95mm_HandSolder, F.Cu at (202.8, 87.8)
- moved K2 70.6 mm to (165.1, 63.5)
- moved K4 30.4 mm to (195.6, 63.5)
Connections:
- K1 pad 1: Net-(K1-Pad1) -> +5V
- K2 pad 1: Net-(K2-Pad1) -> +5V
- K3 pad 1: Net-(K3-Pad1) -> +5V
- K4 pad 1: Net-(K4-Pad1) -> +5V

Commit message: Commit
Parts:
- added C1: 10u, Capacitor_SMD:C_0805_2012Metric_Pad1.18x1.45mm_HandSolder, F.Cu at (160.0, 101.6)
- added C10: 100n, Capacitor_SMD:C_0603_1608Metric_Pad1.08x0.95mm_HandSolder, F.Cu at (181.6, 129.6)
- added C11: 100n, Capacitor_SMD:C_0603_1608Metric_Pad1.08x0.95mm_HandSolder, F.Cu at (194.7, 115.8)
- added C12: 100n, Capacitor_SMD:C_0603_1608Metric_Pad1.08x0.95mm_HandSolder, F.Cu at (190.3, 118.3)
- added C13: 100n, Capacitor_SMD:C_0603_1608Metric_Pad1.08x0.95mm_HandSolder, F.Cu at (168.4, 138.3)
- added C14: 100n, Capacitor_SMD:C_0603_1608Metric_Pad1.08x0.95mm_HandSolder, F.Cu at (181.6, 127.1)
- added C2: 100n, Capacitor_SMD:C_0603_1608Metric_Pad1.08x0.95mm_HandSolder, F.Cu at (160.0, 104.1)
- added C3: 100n, Capacitor_SMD:C_0603_1608Metric_Pad1.08x0.95mm_HandSolder, F.Cu at (164.4, 101.6)
- added C4: 1u, Capacitor_SMD:C_0603_1608Metric_Pad1.08x0.95mm_HandSolder, F.Cu at (164.4, 104.1)
- added C5: 100n, Capacitor_SMD:C_0603_1608Metric_Pad1.08x0.95mm_HandSolder, F.Cu at (168.7, 101.6)
- added C6: 100n, Capacitor_SMD:C_0603_1608Metric_Pad1.08x0.95mm_HandSolder, F.Cu at (176.5, 102.9)
- added C7: 100n, Capacitor_SMD:C_0603_1608Metric_Pad1.08x0.95mm_HandSolder, F.Cu at (181.6, 132.1)
- added C8: 100n, Capacitor_SMD:C_0603_1608Metric_Pad1.08x0.95mm_HandSolder, F.Cu at (159.7, 138.3)
- added C9: 100n, Capacitor_SMD:C_0603_1608Metric_Pad1.08x0.95mm_HandSolder, F.Cu at (172.8, 138.3)
- added FB1: Ferrite_Bead, Resistor_SMD:R_0603_1608Metric_Pad0.98x0.95mm_HandSolder, F.Cu at (176.5, 105.4)
- added J1: FTSH-105-01-F-DV-K, FTSH-105-01-F-DV-K-P:FTSH-105-XX-YYY-DV-K-P, F.Cu at (139.7, 119.4)
- added R10: 1k, Resistor_SMD:R_0603_1608Metric_Pad0.98x0.95mm_HandSolder, F.Cu at (155.4, 138.3)
- added R11: 1k, Resistor_SMD:R_0603_1608Metric_Pad0.98x0.95mm_HandSolder, F.Cu at (190.3, 120.8)
- added R12: 10k, Resistor_SMD:R_0603_1608Metric_Pad0.98x0.95mm_HandSolder, F.Cu at (194.7, 118.3)
- added R13: 10k, Resistor_SMD:R_0603_1608Metric_Pad0.98x0.95mm_HandSolder, F.Cu at (190.3, 123.4)
- added R14: 1k, Resistor_SMD:R_0603_1608Metric_Pad0.98x0.95mm_HandSolder, F.Cu at (186.0, 127.1)
- added R15: 1k, Resistor_SMD:R_0603_1608Metric_Pad0.98x0.95mm_HandSolder, F.Cu at (186.0, 129.6)
- added R16: 10k, Resistor_SMD:R_0603_1608Metric_Pad0.98x0.95mm_HandSolder, F.Cu at (177.1, 138.3)
- added R17: 10k, Resistor_SMD:R_0603_1608Metric_Pad0.98x0.95mm_HandSolder, F.Cu at (190.3, 127.1)
- added R18: 1k, Resistor_SMD:R_0603_1608Metric_Pad0.98x0.95mm_HandSolder, F.Cu at (181.6, 134.6)
- added R19: 1k, Resistor_SMD:R_0603_1608Metric_Pad0.98x0.95mm_HandSolder, F.Cu at (194.7, 120.8)
- added R20: 10k, Resistor_SMD:R_0603_1608Metric_Pad0.98x0.95mm_HandSolder, F.Cu at (194.7, 123.4)
- added R21: 10k, Resistor_SMD:R_0603_1608Metric_Pad0.98x0.95mm_HandSolder, F.Cu at (186.0, 132.1)
- added R5: 10k, Resistor_SMD:R_0603_1608Metric_Pad0.98x0.95mm_HandSolder, F.Cu at (180.9, 102.9)
- added R6: 1k, Resistor_SMD:R_0603_1608Metric_Pad0.98x0.95mm_HandSolder, F.Cu at (137.0, 126.0)
- added R7: 10k, Resistor_SMD:R_0603_1608Metric_Pad0.98x0.95mm_HandSolder, F.Cu at (146.8, 115.7)
- added R8: 1k, Resistor_SMD:R_0603_1608Metric_Pad0.98x0.95mm_HandSolder, F.Cu at (190.3, 115.8)
- added R9: 10k, Resistor_SMD:R_0603_1608Metric_Pad0.98x0.95mm_HandSolder, F.Cu at (164.1, 138.3)
- added S1: 100AWSP1T1B4M2RE, 100AWSP1T1B4M2RE:100AWSP1T1B4M2RE, F.Cu at (217.2, 109.2)
- added S2: 100AWSP1T1B4M2RE, 100AWSP1T1B4M2RE:100AWSP1T1B4M2RE, F.Cu at (217.2, 118.9)
- added S3: 100AWSP1T1B4M2RE, 100AWSP1T1B4M2RE:100AWSP1T1B4M2RE, F.Cu at (233.5, 109.2)
- added S4: 100AWSP1T1B4M2RE, 100AWSP1T1B4M2RE:100AWSP1T1B4M2RE, F.Cu at (217.2, 128.6)
- added S5: 100AWSP1T1B4M2RE, 100AWSP1T1B4M2RE:100AWSP1T1B4M2RE, F.Cu at (233.5, 118.9)
- added S6: 100AWSP1T1B4M2RE, 100AWSP1T1B4M2RE:100AWSP1T1B4M2RE, F.Cu at (249.9, 109.2)
- added S7: 100AWSP1T1B4M2RE, 100AWSP1T1B4M2RE:100AWSP1T1B4M2RE, F.Cu at (233.5, 128.6)
- added S8: 100AWSP1T1B4M2RE, 100AWSP1T1B4M2RE:100AWSP1T1B4M2RE, F.Cu at (249.9, 118.9)
- added U1: STM32L052K6Tx, Package_QFP:LQFP-32_7x7mm_P0.8mm, F.Cu at (144.8, 101.6)
Connections:
- net Net-(Q1-Pad1) renamed /RELAY1_OUT
- net Net-(Q2-Pad1) renamed /RELAY2_OUT
- net Net-(Q3-Pad1) renamed /RELAY3_OUT
- net Net-(Q4-Pad1) renamed /RELAY4_OUT
