File: hardware/PRS.sch (KiCad schematic (older format))
At the start: 4 parts

Commit message: Commit
Parts:
- added D1, D2, D3, D4: MMBD7000HC, Package_TO_SOT_SMD:SOT-23_Handsoldering, symbol Device:D_AAK
- added D5: D_Zener, Diode_SMD:D_SMA_Handsoldering, symbol Device:D_Zener
- added Q1, Q2, Q3, Q4: PMV37ENEA, Package_TO_SOT_SMD:SOT-23_Handsoldering, symbol Device:Q_NMOS_GSD
- added R1, R2, R3, R4: 100k, Resistor_SMD:R_0603_1608Metric_Pad0.98x0.95mm_HandSolder, symbol Device:R
- gave numbers to parts that had none: 4
Connections:
- net labels added: +5V, GND
- wire segments 0 -> 73
Other:
- moved on the sheet: K1, K2, K3, K4

Commit message: Commit
Parts:
- added C1: 10u, Capacitor_SMD:C_0805_2012Metric_Pad1.18x1.45mm_HandSolder, symbol Device:C
- added C10, C11, C12, C13, C14, C2, C3, C5, C6, C7, C8, C9: 100n, Capacitor_SMD:C_0603_1608Metric_Pad1.08x0.95mm_HandSolder, symbol Device:C
- added C4: 1u, Capacitor_SMD:C_0603_1608Metric_Pad1.08x0.95mm_HandSolder, symbol Device:C
- added D?: LED, symbol Device:LED
- added FB1: Ferrite_Bead, Resistor_SMD:R_0603_1608Metric_Pad0.98x0.95mm_HandSolder, symbol Device:Ferrite_Bead
- added J1: FTSH-105-01-F-DV-K, FTSH-105-XX-YYY-DV-K-P, symbol FTSH-105-01-F-DV-K-P:FTSH-105-01-F-DV-K-P
- added Q? (x4): PMV37ENEA, Package_TO_SOT_SMD:SOT-23_Handsoldering, symbol Device:Q_NMOS_GSD
- added R10, R11, R14, R15, R18, R19, R6, R8: 1k, Resistor_SMD:R_0603_1608Metric_Pad0.98x0.95mm_HandSolder, symbol Device:R
- added R12, R13, R16, R17, R20, R21, R5, R7, R9: 10k, Resistor_SMD:R_0603_1608Metric_Pad0.98x0.95mm_HandSolder, symbol Device:R
- added R? (x2): R, symbol Device:R
- added S1, S2, S3, S4, S5, S6, S7, S8: 100AWSP1T1B4M2RE, 100AWSP1T1B4M2RE:100AWSP1T1B4M2RE, symbol 100AWSP1T1B4M2RE:100AWSP1T1B4M2RE
- added U1: STM32L052K6Tx, Package_QFP:LQFP-32_7x7mm_P0.8mm, symbol MCU_ST_STM32L0:STM32L052K6Tx
Connections:
- net labels added: +3.3V, RELAY1_AUTO_MAN, RELAY1_IN, RELAY1_OUT, RELAY2_AUTO_MAN, RELAY2_IN, RELAY2_OUT, RELAY3_AUTO_MAN, RELAY3_IN, RELAY3_OUT, RELAY4_AUTO_MAN, RELAY4_IN, RELAY4_OUT, SWCLK, SWDIO, USB_D+, USB_D-, VDD, VDDA, ~RST
- wire segments 73 -> 221
- no-connect marks 0 -> 3
Other:
- note added: "DEBUG"
- note added: "MCU"
- note added: "RELAYS"
- moved on the sheet: D1, D2, D3, D4, D5, K1, K2, K3, K4, Q1, Q2, Q3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
