File: hardware/PRS_front_panel/PRS_front_panel.kicad_pcb (KiCad board)
At the start: 2 copper layers, 84 parts, among them IC1 74LVC125AD,118, J1 FTSH-105-01-F-DV-K, K1 T9AS1D12-5, K2 T9AS1D12-5, K3 T9AS1D12-5, K4 T9AS1D12-5, Q1 PMV37ENEA, Q2 PMV37ENEA, Q3 PMV37ENEA, Q4 PMV37ENEA, U1 STM32L052K6Tx, U2 MCP1825S-3302E/DB

Commit message: Commit
Parts:
- removed D1, D2, D3, D4: MMBD7000HC, Package_TO_SOT_SMD:SOT-23_Handsoldering
- removed D5: D_Zener, Diode_SMD:D_SMA_Handsoldering
- removed K1, K2, K3, K4: T9AS1D12-5, T9AS1D12-5:T9AS1D125
- removed Q1, Q2, Q3, Q4: PMV37ENEA, Package_TO_SOT_SMD:SOT-23_Handsoldering
- removed R1, R2, R3, R4: 100k, Resistor_SMD:R_0603_1608Metric_Pad0.98x0.95mm_HandSolder
- added J2: 530470610, 530470610:MOLEX_530470610, B.Cu at (215.9, 110.5)
- added J3: 530470410, 530470410:MOLEX_530470410, B.Cu at (213.4, 117.3)
