File: hardware/PRS_front_panel/PRS_front_panel.sch (KiCad schematic (older format))
At the start: 84 parts, among them IC1 74LVC125AD,118, J1 FTSH-105-01-F-DV-K, K1 T9AS1D12-5, K2 T9AS1D12-5, K3 T9AS1D12-5, K4 T9AS1D12-5, Q1 PMV37ENEA, Q2 PMV37ENEA, Q3 PMV37ENEA, Q4 PMV37ENEA, U1 STM32L052K6Tx, U2 MCP1825S-3302E/DB

Commit message: Commit
Parts:
- removed D1, D2, D3, D4: MMBD7000HC, Package_TO_SOT_SMD:SOT-23_Handsoldering, symbol Device:D_AAK
- removed D5: D_Zener, Diode_SMD:D_SMA_Handsoldering, symbol Device:D_Zener
- removed K1, K2, K3, K4: T9AS1D12-5, T9AS1D125, symbol T9AS1D12-5:T9AS1D12-5
- removed Q1, Q2, Q3, Q4: PMV37ENEA, Package_TO_SOT_SMD:SOT-23_Handsoldering, symbol Device:Q_NMOS_GSD
- removed R1, R2, R3, R4: 100k, Resistor_SMD:R_0603_1608Metric_Pad0.98x0.95mm_HandSolder, symbol Device:R
- added J2: 530470610, MOLEX_530470610, symbol 530470610:530470610
- added J3: 530470410, MOLEX_530470410, symbol 530470410:530470410
Other:
- note removed: "RELAYS"
- moved on the sheet: C10, C11, C12, C13, C14, C16, C7, C8, C9, D10, D11, D12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
