File: hardware/PRS_relay_board/PRS_relay_board.kicad_pcb (KiCad board)
At the start: 4 copper layers, 160 x 135 mm, 110 parts, among them J1 691313410004, J2 691313410004, J3 UJ2-BH-2-TH, J4 FTSH-105-01-F-DV-K-P, J5 10-32-1031, J6 B3B-XH-A, K1 1-1393210-3, K2 1-1393210-3, K3 1-1393210-3, K4 1-1393210-3, Q1 PMV37ENEA, Q2 PMV37ENEA, Q3 PMV37ENEA, Q4 PMV37ENEA, Q5 BC848, Q6 PMV37ENEA, U1 STCN75, U2 STM32L062K8Tx, U3 74LVC125AD,118, U4 USBLC6-2SC6, U5 UA78M33CKVURG3

Commit message: Change C13 footprint
Parts:
- C13: footprint Capacitor_SMD:C_0805_2012Metric_Pad1.18x1.45mm_HandSolder -> Capacitor_SMD:C_1206_3216Metric_Pad1.33x1.80mm_HandSolder
Changed lines of the file:
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@@
+    )
+  )
+  (module Capacitor_SMD:C_1206_3216Metric_Pad1.33x1.80mm_HandSolder (layer F.Cu)
+    (at 188.82 148.68)
+    (descr "Capacitor SMD 1206 (3216 Metric), square (rectangular) end terminal, IPC_7351 nominal with elongated pad for handsoldering. (Body size source: IPC-SM-782 page 76, https://www.pcb-3d.com/wordpress/wp-content/uploads/ipc-sm-782a_amendment_1_and_2.pdf), generated with kicad-footprint-generator")
+    (tags "capacitor handsolder")
+    (attr smd)
+    (fp_text reference C13 (at 0 -1.85) (layer F.SilkS)
+      (effects (font (size 1 1) (thickness 0.15)))
+    )
+    (fp_text value 10u (at 0 1.85) (layer F.Fab)
+      (effects (font (size 1 1) (thickness 0.15)))
+    )
+    (fp_text user %R (at 0 0) (layer F.Fab)
+      (effects (font (size 0.8 0.8) (thickness 0.12)))
+    )
+    (fp_line (start -1.6 0.8) (end -1.6 -0.8) (layer F.Fab) (width 0.1))
+    (fp_line (start -1.6 -0.8) (end 1.6 -0.8) (layer F.Fab) (width 0.1))
+    (fp_line (start 1.6 -0.8) (end 1.6 0.8) (layer F.Fab) (width 0.1))
+    (fp_line (start 1.6 0.8) (end -1.6 0.8) (layer F.Fab) (width 0.1))
+    (fp_line (start -0.711252 -0.91) (end 0.711252 -0.91) (layer F.SilkS) (width 0.12))
+    (fp_line (start -0.711252 0.91) (end 0.711252 0.91) (layer F.SilkS) (width 0.12))
+    (fp_line (start -2.48 1.15) (end -2.48 -1.15) (layer F.CrtYd) (width 0.05))
+    (fp_line (start -2.48 -1.15) (end 2.48 -1.15) (layer F.CrtYd) (width 0.05))
+    (fp_line (start 2.48 -1.15) (end 2.48 1.15) (layer F.CrtYd) (width 0.05))
+    (fp_line (start 2.48 1.15) (end -2.48 1.15) (layer F.CrtYd) (width 0.05))
+    (pad 2 smd roundrect (at 1.5625 0) (size 1.325 1.8) (layers F.Cu F.Paste F.Mask) (roundrect_rratio 0.188679)
+      (net 10 GND))
+    (pad 1 smd roundrect (at -1.5625 0) (size 1.325 1.8) (layers F.Cu F.Paste F.Mask) (roundrect_rratio 0.188679)
+      (net 13 +3V3))
+    (model ${KISYS3DMOD}/Capacitor_SMD.3dshapes/C_1206_3216Metric.wrl
+      (at (xyz 0 0 0))
+      (scale (xyz 1 1 1))
+      (rotate (xyz 0 0 0))
     )
   )
@@
       (at (xyz 0 0 0))
       (scale (xyz 1 1 1))
-      (rotate (xyz 0 0 0))
-    )
-  )
-  (module Capacitor_SMD:C_0805_2012Metric_Pad1.18x1.45mm_HandSolder (layer F.Cu)
-    (at 188.82 148.68)
-    (descr "Capacitor SMD 0805 (2012 Metric), square (rectangular) end terminal, IPC_7351 nominal with elongated pad for handsoldering. (Body size source: IPC-SM-782 page 76, https://www.pcb-3d.com/wordpress/wp-content/uploads/ipc-sm-782a_amendment_1_and_2.pdf, https://docs.google.com/spreadsheets/d/1BsfQQcO9C6DZCsRaXUlFlo91Tg2WpOkGARC1WS5S8t0/edit?usp=sharing), generated with kicad-footprint-generator")
-    (tags "capacitor handsolder")
-    (attr smd)
-    (fp_text reference C13 (at 0 -1.68) (layer F.SilkS)
-      (effects (font (size 1 1) (thickness 0.15)))
-    )
-    (fp_text value 10u (at 0 1.68) (layer F.Fab)
-      (effects (font (size 1 1) (thickness 0.15)))
-    )
-    (fp_line (start 1.88 0.98) (end -1.88 0.98) (layer F.CrtYd) (width 0.05))
-    (fp_line (start 1.88 -0.98) (end 1.88 0.98) (layer F.CrtYd) (width 0.05))
-    (fp_line (start -1.88 -0.98) (end 1.88 -0.98) (layer F.CrtYd) (width 0.05))
-    (fp_line (start -1.88 0.98) (end -1.88 -0.98) (layer F.CrtYd) (width 0.05))
-    (fp_line (start -0.261252 0.735) (end 0.261252 0.735) (layer F.SilkS) (width 0.12))
-    (fp_line (start -0.261252 -0.735) (end 0.261252 -0.735) (layer F.SilkS) (width 0.12))
-    (fp_line (start 1 0.625) (end -1 0.625) (layer F.Fab) (width 0.1))
-    (fp_line (start 1 -0.625) (end 1 0.625) (layer F.Fab) (width 0.1))
-    (fp_line (start -1 -0.625) (end 1 -0.625) (layer F.Fab) (width 0.1))
-    (fp_line (start -1 0.625) (end -1 -0.625) (layer F.Fab) (width 0.1))
-    (fp_text user %R (at 0 0) (layer F.Fab)
-      (effects (font (size 0.5 0.5) (thickness 0.08)))
-    )
-    (pad 2 smd roundrect (at 1.0375 0) (size 1.175 1.45) (layers F.Cu F.Paste F.Mask) (roundrect_rratio 0.212766)
-      (net 10 GND))
-    (pad 1 smd roundrect (at -1.0375 0) (size 1.175 1.45) (layers F.Cu F.Paste F.Mask) (roundrect_rratio 0.212766)
-      (net 13 +3V3))
-    (model ${KISYS3DMOD}/Capacitor_SMD.3dshapes/C_0805_2012Metric.wrl
-      (at (xyz 0 0 0))
-      (scale (xyz 1 1 1))

Commit message: Create PCB Layout
Parts:
- R13, R14, R15, R25, R26, R27, R32, R5: value 330R -> 220R
- moved J5 348.5 mm to (68.0, 132.9), turned to 270 degrees
- moved PS1 284.2 mm to (80.0, 128.0)
- moved C5 268.9 mm to (147.0, 133.0), turned to 90 degrees
- moved C3 238.8 mm to (135.0, 135.0), turned to 270 degrees
- moved R6 234.9 mm to (80.0, 162.5), turned to 180 degrees
- moved R43 225.1 mm to (130.0, 72.0), turned to 90 degrees
- moved R41 221.0 mm to (131.5, 84.5), turned to 270 degrees
- moved R42 220.4 mm to (131.5, 72.0), turned to 270 degrees
- moved D9 219.0 mm to (135.0, 71.5), turned to 90 degrees
- moved U5 218.8 mm to (141.0, 134.0), turned to 90 degrees
- moved C19 216.3 mm to (127.3, 96.7), turned to 270 degrees
- moved LED1 214.3 mm to (96.0, 180.5)
- moved R40 214.2 mm to (131.5, 78.5), turned to 270 degrees
- moved Q6 211.0 mm to (135.0, 78.0), turned to 90 degrees
- moved D7 207.7 mm to (72.0, 106.0), turned to 180 degrees
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Connections:
- net Net-(J5-Pad1) renamed /Power/N
- net Net-(J5-Pad3) renamed /Power/L
- J1 pad 1: /Relays/RELAY1_COM -> /Relays/RELAY2_COM
- J1 pad 2: /Relays/RELAY1_NO -> /Relays/RELAY2_NO
- J1 pad 3: /Relays/RELAY2_COM -> /Relays/RELAY1_COM
- J1 pad 4: /Relays/RELAY2_NO -> /Relays/RELAY1_NO
- J2 pad 1: /Relays/RELAY3_COM -> /Relays/RELAY4_COM
- J2 pad 2: /Relays/RELAY3_NO -> /Relays/RELAY4_NO
- J2 pad 3: /Relays/RELAY4_COM -> /Relays/RELAY3_COM
- J2 pad 4: /Relays/RELAY4_NO -> /Relays/RELAY3_NO
- J6 pad 1: +12V -> Net-(J6-Pad1)
- J6 pad 2: Net-(J6-Pad2) -> +12V
- K1 pad A2: Net-(D6-Pad1) -> Net-(D2-Pad1)
- K1 pad C: /Relays/RELAY2_COM -> /Relays/RELAY1_COM
- K1 pad NO: /Relays/RELAY2_NO -> /Relays/RELAY1_NO
- K2 pad A2: Net-(D2-Pad1) -> Net-(D4-Pad1)
- K2 pad C: /Relays/RELAY1_COM -> /Relays/RELAY2_COM
- K2 pad NO: /Relays/RELAY1_NO -> /Relays/RELAY2_NO
- K3 pad A2: Net-(D8-Pad1) -> Net-(D6-Pad1)
- K3 pad C: /Relays/RELAY4_COM -> /Relays/RELAY3_COM
- K3 pad NO: /Relays/RELAY4_NO -> /Relays/RELAY3_NO
- K4 pad A2: Net-(D4-Pad1) -> Net-(D8-Pad1)
- K4 pad C: /Relays/RELAY3_COM -> /Relays/RELAY4_COM
- K4 pad NO: /Relays/RELAY3_NO -> /Relays/RELAY4_NO
- LED3 pad 4: Net-(LED3-Pad4) -> GND
- Q1 pad 1: /Front Panel/RELAY3_OUT -> /Front Panel/RELAY1_OUT
- Q1 pad 3: Net-(D6-Pad1) -> Net-(D2-Pad1)
- Q2 pad 1: /Front Panel/RELAY1_OUT -> /Front Panel/RELAY2_OUT
- Q2 pad 3: Net-(D2-Pad1) -> Net-(D4-Pad1)
- Q3 pad 1: /Front Panel/RELAY4_OUT -> /Front Panel/RELAY3_OUT
- Q3 pad 3: Net-(D8-Pad1) -> Net-(D6-Pad1)
- Q4 pad 1: /Front Panel/RELAY2_OUT -> /Front Panel/RELAY4_OUT
- Q4 pad 3: Net-(D4-Pad1) -> Net-(D8-Pad1)
- R20 pad 2: /Front Panel/RELAY4_OUT -> /Front Panel/RELAY2_OUT
- R21 pad 2: /Front Panel/RELAY3_OUT -> /Front Panel/RELAY1_OUT
- R22 pad 2: /Front Panel/RELAY2_OUT -> /Front Panel/RELAY3_OUT
- R23 pad 2: /Front Panel/RELAY1_OUT -> /Front Panel/RELAY4_OUT
- R42 pad 1: Net-(J6-Pad2) -> Net-(J6-Pad1)
- U2 pad 10: /Front Panel/RELAY3_IN -> /Front Panel/RELAY3_USB_MAN
- U2 pad 11: /Front Panel/RELAY3_USB_MAN -> /Front Panel/RELAY3_IN
- U2 pad 12: /Front Panel/RELAY4_IN -> /Front Panel/RELAY4_USB_MAN
- U2 pad 13: /Front Panel/RELAY4_USB_MAN -> /Front Panel/RELAY4_IN
- U2 pad 6: /Front Panel/RELAY1_IN -> /Front Panel/RELAY1_USB_MAN
- U2 pad 7: /Front Panel/RELAY1_USB_MAN -> /Front Panel/RELAY1_IN
- U2 pad 8: /Front Panel/RELAY2_IN -> /Front Panel/RELAY2_USB_MAN
- U2 pad 9: /Front Panel/RELAY2_USB_MAN -> /Front Panel/RELAY2_IN
Routing:
- net /Front Panel/RELAY4_OUT: track 0.00 -> 127.4 mm, vias 0 -> 3
- net /Front Panel/RELAY3_OUT: track 0.00 -> 103.0 mm, vias 0 -> 3
- net /Sheet6168966E/1Y: track 95.1 -> 0.00 mm
- net /MCU/VBUS_SENSE: track 0.00 -> 95.1 mm
- net /Front Panel/RELAY1_USB_MAN: track 0.00 -> 93.5 mm
- net /MCU/USB_D-: track 0.00 -> 93.2 mm
- net /MCU/USB_D+: track 0.00 -> 92.4 mm
- net /Cooling/FAN_TACH: track 0.00 -> 84.9 mm
- net /Front Panel/1Y: track 0.00 -> 83.3 mm
- net /Front Panel/RELAY1_IN: track 0.00 -> 82.6 mm
- net /Relays/RELAY2_COM: track 0.00 -> 78.7 mm
- net /Relays/RELAY3_NO: track 0.00 -> 76.8 mm
- net +12V: track 0.00 -> 75.0 mm, vias 0 -> 1
- net /Relays/RELAY3_COM: track 0.00 -> 69.7 mm
- net /Front Panel/RELAY2_OUT: track 0.00 -> 69.6 mm, vias 0 -> 4
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- added copper zone on PWR, net +12V
- added copper zone on F.Cu, net +3V3
- added copper zone on PWR, net +3V3
- added copper zone on F.Cu, net GND
- added copper zone on GND, net GND
Other:
- net class Default: clearance 0.2 -> 0.1; trace_width 0.25 -> 0.35
- net class RELAY added: clearance 1, trace_width 4, via_dia 0.8, via_drill 0.4
- rule trace_clearance: 0.2 -> 0.1
- board text added: "Designed by: Priit Tänav github.com/prtana/power-relay-switcher"
- board text added: "Power Relay Switcher 1.0"

Commit message: Commit
Parts:
- added R44: 10k, Resistor_SMD:R_0603_1608Metric_Pad0.98x0.95mm_HandSolder, F.Cu at (131.5, 72.0)
- added RV1: ERZE11A431, Varistor:RV_Disc_D12mm_W6.3mm_P7.5mm, F.Cu at (176.3, 63.0)
- added RV2: ERZE11A431, Varistor:RV_Disc_D12mm_W6.3mm_P7.5mm, F.Cu at (161.0, 63.0)
- added RV3: ERZE11A431, Varistor:RV_Disc_D12mm_W6.3mm_P7.5mm, F.Cu at (90.3, 63.0)
- added RV4: ERZE11A431, Varistor:RV_Disc_D12mm_W6.3mm_P7.5mm, F.Cu at (75.0, 63.0)
- moved H3 27.0 mm to (65.0, 153.0)
- moved H2 9.49 mm to (212.0, 64.0)
- moved H4 9.49 mm to (212.0, 171.0)
- moved LED2 8.14 mm to (124.5, 181.5)
- moved R14 8.14 mm to (124.5, 174.5)
- moved R15 8.14 mm to (127.0, 174.5)
- moved LED1 8.06 mm to (88.0, 181.5)
- moved LED3 8.06 mm to (161.0, 181.5)
- moved LED4 8.06 mm to (197.5, 181.5)
- moved R13 8.06 mm to (90.5, 174.5)
- moved R25 8.06 mm to (161.0, 174.5)
- moved R26 8.06 mm to (163.5, 174.5)
- moved R27 8.06 mm to (197.5, 174.5)
- moved R32 8.06 mm to (200.0, 174.5)
- moved R5 8.06 mm to (88.0, 174.5)
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Connections:
- J6 pad 1: Net-(J6-Pad1) -> +12V
- J6 pad 2: +12V -> Net-(D9-Pad1)
- J6 pad 3: Net-(D9-Pad1) -> Net-(J6-Pad3)
- R42 pad 1: Net-(J6-Pad1) -> Net-(J6-Pad3)
Routing:
- net Net-(J6-Pad3): track 0.00 -> 17.7 mm
- net +12V: track 75.0 -> 63.3 mm, vias 1 -> 2
- net Net-(J6-Pad1): track 11.2 -> 0.00 mm
- net /Front Panel/RELAY2_IN: track 45.0 -> 55.5 mm
- net /Front Panel/RELAY2_USB_MAN: track 60.3 -> 69.9 mm
- net /Front Panel/RELAY1_IN: track 82.6 -> 91.9 mm
- net /Front Panel/RELAY1_USB_MAN: track 93.5 -> 102.1 mm
- net /Relays/RELAY1_NO: track 48.9 -> 57.4 mm
- net /Front Panel/RELAY3_OUT: track 103.0 -> 95.4 mm
- net /Front Panel/RELAY4_USB_MAN: track 49.8 -> 42.3 mm
- net /Front Panel/RELAY4_IN: track 59.4 -> 52.8 mm
- net /Front Panel/RELAY2_OUT: track 69.6 -> 76.3 mm
- net /Front Panel/RELAY1_OUT: track 68.0 -> 74.3 mm
- net /Relays/RELAY4_NO: track 50.0 -> 56.0 mm
- net /Relays/RELAY4_COM: track 54.6 -> 60.6 mm
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- added copper zone on F.Cu, net +12V
Other:
- board size 160 x 135 mm -> 160 x 137 mm
- net class Default: clearance 0.1 -> 0.2
- rule trace_clearance: 0.1 -> 0.2
