File: hardware/PRS_relay_board/KiCad/MCU.kicad_sch (KiCad schematic)
At the start: 19 parts, among them J3 UJ2-BH-2-TH, J4 FTSH-105-01-F-DV-K-P, U2 STM32L062K8Tx, U4 USBLC6-2SC6

Commit message: Commit
Parts:
- C13: renamed from C?; value (none) -> 10u; footprint (none) -> Capacitor_SMD:C_1206_3216Metric_Pad1.33x1.80mm_HandSolder
- C14, C15, C18, C4, C8: renamed from C?; value (none) -> 100n; footprint (none) -> Capacitor_SMD:C_0603_1608Metric_Pad1.08x0.95mm_HandSolder
- C17: renamed from C?; value (none) -> 1u; footprint (none) -> Capacitor_SMD:C_0603_1608Metric_Pad1.08x0.95mm_HandSolder
- FB1: renamed from FB?; value (none) -> BLM18HE601SN1D; footprint (none) -> Resistor_SMD:R_0603_1608Metric_Pad0.98x0.95mm_HandSolder
- R10, R11: renamed from R?; value (none) -> 100k; footprint (none) -> Resistor_SMD:R_0603_1608Metric_Pad0.98x0.95mm_HandSolder
- R20, R21, R22, R23: renamed from R?; value (none) -> 100R; footprint (none) -> Resistor_SMD:R_0603_1608Metric_Pad0.98x0.95mm_HandSolder
- R24: renamed from R?; value (none) -> 10k; footprint (none) -> Resistor_SMD:R_0603_1608Metric_Pad0.98x0.95mm_HandSolder
