File: hardware/PRS_relay_board/KiCad/front_panel.kicad_sch (KiCad schematic)
At the start: 46 parts

Commit message: Commit
Parts:
- C1, C10, C11, C12, C16, C2, C6, C7, C9: renamed from C?; value (none) -> 100n; footprint (none) -> Capacitor_SMD:C_0603_1608Metric_Pad1.08x0.95mm_HandSolder
- LED1, LED2, LED3, LED4: renamed from LED?; value (none) -> 553-0122F; footprint (none) -> 553-0122:5530122F
- R12, R18, R19, R30, R31, R35, R36, R8: renamed from R?; value (none) -> 10k; footprint (none) -> Resistor_SMD:R_0603_1608Metric_Pad0.98x0.95mm_HandSolder
- R13, R14, R15, R25, R26, R27, R32, R5: renamed from R?; value (none) -> 220R; footprint (none) -> Resistor_SMD:R_0603_1608Metric_Pad0.98x0.95mm_HandSolder
- R16, R17, R28, R29, R33, R34, R6, R7: renamed from R?; value (none) -> 1k; footprint (none) -> Resistor_SMD:R_0603_1608Metric_Pad0.98x0.95mm_HandSolder
- S1, S2, S3, S4, S5, S6, S7, S8: renamed from S?; value (none) -> 100SP1T2B4M7RE; footprint (none) -> 100SP1T2B4M7RE:100SP1T2B4M7RE
- U3: renamed from IC?; value (none) -> 74LVC125AD,118; footprint (none) -> 74LVC125AD,118:SOIC127P600X175-14N
