File: hardware/PRS_relay_board/KiCad/power.kicad_sch (KiCad schematic)
At the start: 5 parts

Commit message: Commit
Parts:
- C3: renamed from C?; value (none) -> 330n; footprint (none) -> Capacitor_SMD:C_0603_1608Metric_Pad1.08x0.95mm_HandSolder
- C5: renamed from C?; value (none) -> 100n; footprint (none) -> Capacitor_SMD:C_0603_1608Metric_Pad1.08x0.95mm_HandSolder
- J5: renamed from J?; value (none) -> 10-32-1031; footprint (none) -> 10-32-1031:SHDR3W114P0X508_1X3_1416X1140X1425P
- PS1: renamed from PS?; value (none) -> RAC10-12SK_277; footprint (none) -> RAC10-12SK_277:RAC10-12SK_277
- U5: renamed from IC?; value (none) -> UA78M33CKVURG3; footprint (none) -> UA78M33CKVURG3:TPS7A6533QKVURQ1
Changed lines of the file:
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@@
   (symbol (lib_id "power:GND") (at 119.38 85.09 0) (unit 1)
     (in_bom yes) (on_board yes)
-    (property "Reference" "#PWR?" (id 0) (at 119.38 91.44 0)
-      (effects (font (size 1.27 1.27)) hide)
-    )
-    (property "Value" "" (id 1) (at 119.507 89.4842 0))
+    (property "Reference" "#PWR014" (id 0) (at 119.38 91.44 0)
+      (effects (font (size 1.27 1.27)) hide)
+    )
+    (property "Value" "GND" (id 1) (at 119.507 89.4842 0))
     (property "Footprint" "" (id 2) (at 119.38 85.09 0)
       (effects (font (size 1.27 1.27)) hide)
@@
   (symbol (lib_id "power:+12V") (at 119.38 77.47 0) (unit 1)
     (in_bom yes) (on_board yes)
-    (property "Reference" "#PWR?" (id 0) (at 119.38 81.28 0)
-      (effects (font (size 1.27 1.27)) hide)
-    )
-    (property "Value" "" (id 1) (at 119.761 73.0758 0))
+    (property "Reference" "#PWR09" (id 0) (at 119.38 81.28 0)
+      (effects (font (size 1.27 1.27)) hide)
+    )
+    (property "Value" "+12V" (id 1) (at 119.761 73.0758 0))
     (property "Footprint" "" (id 2) (at 119.38 77.47 0)
       (effects (font (size 1.27 1.27)) hide)
@@
   (symbol (lib_id "RAC10-12SK_277:RAC10-12SK_277") (at 78.74 80.01 0) (unit 1)
     (in_bom yes) (on_board yes)
-    (property "Reference" "PS?" (id 0) (at 97.79 73.279 0))
-    (property "Value" "" (id 1) (at 97.79 75.5904 0))
-    (property "Footprint" "" (id 2) (at 113.03 77.47 0)
+    (property "Reference" "PS1" (id 0) (at 97.79 73.279 0))
+    (property "Value" "RAC10-12SK_277" (id 1) (at 97.79 75.5904 0))
+    (property "Footprint" "RAC10-12SK_277:RAC10-12SK_277" (id 2) (at 113.03 77.47 0)
       (effects (font (size 1.27 1.27)) (justify left) hide)
     )
@@
   (symbol (lib_id "10-32-1031:10-32-1031") (at 73.66 78.74 0) (mirror y) (unit 1)
     (in_bom yes) (on_board yes)
-    (property "Reference" "J?" (id 0) (at 66.2432 72.009 0))
-    (property "Value" "" (id 1) (at 66.2432 74.3204 0))
-    (property "Footprint" "" (id 2) (at 57.15 76.2 0)
+    (property "Reference" "J5" (id 0) (at 66.2432 72.009 0))
+    (property "Value" "10-32-1031" (id 1) (at 66.2432 74.3204 0))
+    (property "Footprint" "10-32-1031:SHDR3W114P0X508_1X3_1416X1140X1425P" (id 2) (at 57.15 76.2 0)
       (effects (font (size 1.27 1.27)) (justify left) hide)
     )
@@
   (symbol (lib_id "Device:C") (at 181.61 88.9 0) (unit 1)
     (in_bom yes) (on_board yes)
-    (property "Reference" "C?" (id 0) (at 184.531 87.7316 0)
-      (effects (font (size 1.27 1.27)) (justify left))
-    )
-    (property "Value" "" (id 1) (at 184.531 90.043 0)
-      (effects (font (size 1.27 1.27)) (justify left))
-    )
-    (property "Footprint" "" (id 2) (at 182.5752 92.71 0)
+    (property "Reference" "C3" (id 0) (at 184.531 87.7316 0)
+      (effects (font (size 1.27 1.27)) (justify left))
+    )
+    (property "Value" "330n" (id 1) (at 184.531 90.043 0)
+      (effects (font (size 1.27 1.27)) (justify left))
+    )
+    (property "Footprint" "Capacitor_SMD:C_0603_1608Metric_Pad1.08x0.95mm_HandSolder" (id 2) (at 182.5752 92.71 0)
       (effects (font (size 1.27 1.27)) hide)
     )
@@
   (symbol (lib_id "Device:C") (at 200.66 91.44 0) (unit 1)
     (in_bom yes) (on_board yes)
-    (property "Reference" "C?" (id 0) (at 203.581 90.2716 0)
-      (effects (font (size 1.27 1.27)) (justify left))
-    )
-    (property "Value" "" (id 1) (at 203.581 92.583 0)
-      (effects (font (size 1.27 1.27)) (justify left))
-    )
-    (property "Footprint" "" (id 2) (at 201.6252 95.25 0)
+    (property "Reference" "C5" (id 0) (at 203.581 90.2716 0)
+      (effects (font (size 1.27 1.27)) (justify left))
+    )
+    (property "Value" "100n" (id 1) (at 203.581 92.583 0)
+      (effects (font (size 1.27 1.27)) (justify left))
+    )
+    (property "Footprint" "Capacitor_SMD:C_0603_1608Metric_Pad1.08x0.95mm_HandSolder" (id 2) (at 201.6252 95.25 0)
       (effects (font (size 1.27 1.27)) hide)
     )
@@
   (symbol (lib_id "power:GND") (at 231.14 85.09 0) (unit 1)
     (in_bom yes) (on_board yes)
-    (property "Reference" "#PWR?" (id 0) (at 231.14 91.44 0)
-      (effects (font (size 1.27 1.27)) hide)
-    )
-    (property "Value" "" (id 1) (at 231.267 89.4842 0))
+    (property "Reference" "#PWR038" (id 0) (at 231.14 91.44 0)
+      (effects (font (size 1.27 1.27)) hide)
+    )
+    (property "Value" "GND" (id 1) (at 231.267 89.4842 0))
     (property "Footprint" "" (id 2) (at 231.14 85.09 0)
       (effects (font (size 1.27 1.27)) hide)
@@
   (symbol (lib_id "power:GND") (at 181.61 95.25 0) (unit 1)
     (in_bom yes) (on_board yes)
-    (property "Reference" "#PWR?" (id 0) (at 181.61 101.6 0)
-      (effects (font (size 1.27 1.27)) hide)
-    )
-    (property "Value" "" (id 1) (at 181.737 99.6442 0))
+    (property "Reference" "#PWR027" (id 0) (at 181.61 101.6 0)
+      (effects (font (size 1.27 1.27)) hide)
+    )
+    (property "Value" "GND" (id 1) (at 181.737 99.6442 0))
     (property "Footprint" "" (id 2) (at 181.61 95.25 0)
       (effects (font (size 1.27 1.27)) hide)
@@
   (symbol (lib_id "power:GND") (at 200.66 97.79 0) (unit 1)
     (in_bom yes) (on_board yes)
-    (property "Reference" "#PWR?" (id 0) (at 200.66 104.14 0)
-      (effects (font (size 1.27 1.27)) hide)
-    )
-    (property "Value" "" (id 1) (at 200.787 102.1842 0))
+    (property "Reference" "#PWR033" (id 0) (at 200.66 104.14 0)
+      (effects (font (size 1.27 1.27)) hide)
+    )
+    (property "Value" "GND" (id 1) (at 200.787 102.1842 0))
     (property "Footprint" "" (id 2) (at 200.66 97.79 0)
       (effects (font (size 1.27 1.27)) hide)
@@
   (symbol (lib_id "PRS_relay_board-rescue:+3.3V-power") (at 200.66 77.47 0) (unit 1)
     (in_bom yes) (on_board yes)
-    (property "Reference" "#PWR?" (id 0) (at 200.66 81.28 0)
-      (effects (font (size 1.27 1.27)) hide)
-    )
-    (property "Value" "" (id 1) (at 201.041 73.0758 0))
+    (property "Reference" "#PWR031" (id 0) (at 200.66 81.28 0)
+      (effects (font (size 1.27 1.27)) hide)
+    )
+    (property "Value" "+3.3V" (id 1) (at 201.041 73.0758 0))
     (property "Footprint" "" (id 2) (at 200.66 77.47 0)
       (effects (font (size 1.27 1.27)) hide)
@@
   (symbol (lib_id "UA78M33CKVURG3:UA78M33CKVURG3") (at 203.2 82.55 0) (unit 1)
     (in_bom yes) (on_board yes)
-    (property "Reference" "IC?" (id 0) (at 215.9 75.819 0))
-    (property "Value" "" (id 1) (at 215.9 78.1304 0))
-    (property "Footprint" "" (id 2) (at 224.79 80.01 0)
+    (property "Reference" "U5" (id 0) (at 215.9 75.819 0))
+    (property "Value" "UA78M33CKVURG3" (id 1) (at 215.9 78.1304 0))
+    (property "Footprint" "UA78M33CKVURG3:TPS7A6533QKVURQ1" (id 2) (at 224.79 80.01 0)
       (effects (font (size 1.27 1.27)) (justify left) hide)
     )
@@
   (symbol (lib_id "power:+12V") (at 181.61 80.01 0) (unit 1)
     (in_bom yes) (on_board yes)
-    (property "Reference" "#PWR?" (id 0) (at 181.61 83.82 0)
-      (effects (font (size 1.27 1.27)) hide)
-    )
-    (property "Value" "" (id 1) (at 181.991 75.6158 0))
+    (property "Reference" "#PWR026" (id 0) (at 181.61 83.82 0)
+      (effects (font (size 1.27 1.27)) hide)
+    )
+    (property "Value" "+12V" (id 1) (at 181.991 75.6158 0))
     (property "Footprint" "" (id 2) (at 181.61 80.01 0)
       (effects (font (size 1.27 1.27)) hide)
