File: hardware/PRS_relay_board/KiCad/relays.kicad_sch (KiCad schematic)
At the start: 26 parts

Commit message: Commit
Parts:
- D1, D3, D5, D7: renamed from D?; value (none) -> MM3Z24VST1G; footprint (none) -> Diode_SMD:D_SOD-323
- D2, D4, D6, D8: renamed from D?; value (none) -> MMBD7000HC; footprint (none) -> Package_TO_SOT_SMD:SOT-23_Handsoldering
- J1, J2: renamed from J?; value (none) -> 691313410004; footprint (none) -> 691313410004:691313410004
- K1, K2, K3, K4: renamed from K?; value (none) -> 1-1393210-3; footprint (none) -> T9AS1D12-12:TE_1-1393210-3
- Q1, Q2, Q3, Q4: renamed from Q?; value (none) -> PMV37ENEA; footprint (none) -> Package_TO_SOT_SMD:SOT-23_Handsoldering
- R1, R2, R3, R4: renamed from R?; value (none) -> 100k; footprint (none) -> Resistor_SMD:R_0603_1608Metric_Pad0.98x0.95mm_HandSolder
